Commit message: add new urdf
Signed-off-by: alan Zhang <zhj.buffer@gmail.com>

File: yhs_chassis_description/src/urdf/amr_scan.urdf (robot description, URDF)
Before this commit: robot yhs_chassis_description, 13 links, 12 joints
Links:
- link base_link: geometry collision box size=0.6 0.4 0.4; visual mesh filename=package://yhs_chassis_description/meshes/DGT-001M.STL
